File: hub_pcb/FRCHubController/FRCHubController.kicad_sch (KiCad schematic)
At the start: 8 parts, among them J1 Conn_01x03_Socket, J2 Conn_01x03_Socket, J3 Conn_01x03_Socket, J4 Barrel_Jack_Switch_Pin3Ring, J5 Conn_02x08_Odd_Even, U6 TXB0102DCU

Commit message: Layout PCB
Connections:
- net B2: now also U1.15 (GPIO37)
- net LED: now also U1.25 (GPIO1); no longer U1.15 (GPIO37)
Changed lines of the file:
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@@
 	(wire
 		(pts
+			(xy 139.7 62.23) (xy 154.94 62.23)
+		)
+		(stroke
+			(width 0)
+			(type default)
+		)
+	)
+	(wire
+		(pts
 			(xy 34.29 101.6) (xy 26.67 101.6)
 		)
@@
 		)
 	)
+	(label "LED"
+		(at 139.7 62.23 0)
+		(effects
+			(font
+				(size 1.27 1.27)
+			)
+			(justify left bottom)
+		)
+	)
 	(label "R1"
 		(at 193.04 44.45 180)
@@
 		)
 	)
+	(label "B2"
+		(at 193.04 59.69 180)
+		(effects
+			(font
+				(size 1.27 1.27)
+			)
+			(justify right bottom)
+		)
+	)
 	(label "PWM2"
 		(at 181.61 123.19 0)
@@
 		)
 	)
-	(label "LED"
-		(at 193.04 59.69 180)
-		(effects
-			(font
-				(size 1.27 1.27)
-			)
-			(justify right bottom)
-		)
-	)

Commit message: Complete layout
Parts:
- added H1, H2, H3, H4: MountingHole_Pad, MountingHole:MountingHole_5.3mm_M5_Pad, symbol Mechanical:MountingHole_Pad
- added J6: Screw_Terminal_01x02, 282815-2:TE_282815-2, symbol Connector:Screw_Terminal_01x02
Connections:
- net +12V: now also J6.1 (Pin_1)
- net GND: now also H1.1, H2.1, H3.1, H4.1, J6.2 (Pin_2)
Other:
- note added: "12V Connection"
- note added: "Mounting holes"
- moved on the sheet: J2, J3, R1, U6
