File: hub_pcb/FRCHubController/photoeye.kicad_sch (KiCad schematic)
At the start: 3 parts

Commit message: Complete layout
Parts:
- removed U2: ~, Library:M12, symbol FRCHubController:M12_4_Pin_Male
- added U2: Conn_01x05_Socket, Library:M12, symbol Connector:Conn_01x05_Socket
Connections:
- net +12V: now also U2.1 (Pin_1)
- net GND: now also U2.3 (Pin_3)
- net at R4.2: now also U2.4 (Pin_4)
- no-connect marks 1 -> 2
Other:
- moved on the sheet: R3, R4
